File: electrical/WRO_RevB_2/WRO_RevB_2.kicad_pcb (KiCad board)
At the start: 2 copper layers, 117.5 x 50.6 mm, 25 parts, among them J11 MOTOR, J2 Conn_01x04_Pin, J3 Conn_01x04_Pin, J4 Conn_01x11_Pin, J5 Conn_01x08_Pin, U2 ROB-14450

Commit message: Revert "Merge branch 'main' of https://github.com/Nakashima26/WRO_FE_2026_FoxRobotics"
This reverts commit 232f9ecb01216201165b5abf43ae09e229c3eea8, reversing
changes made to 212c0f9856f89e84f48e320d89d4fd8fc24ab9e3.
Parts:
- moved J11 20.2 mm to (141.1, 91.5), turned to 180 degrees
- moved US1 15.0 mm to (154.0, 91.1)
- moved R4 13.9 mm to (133.5, 85.0), turned to 90 degrees
- moved US3 13.8 mm to (154.0, 105.2)
- moved G*** 9.55 mm to (162.3, 83.5)
- moved R3 9.47 mm to (137.4, 85.0), turned to 90 degrees
- moved C5 6.12 mm to (133.9, 114.7)
- moved C6 6.12 mm to (139.9, 115.7)
- moved TOF3 4.70 mm to (140.3, 98.1)
- moved TOF4 4.59 mm to (140.3, 105.2)
- moved TOF1 4.00 mm to (128.8, 98.1)
- moved TOF2 3.87 mm to (128.8, 105.2)
- moved US2 2.74 mm to (154.0, 98.1)
Routing:
- net GND: track 26.2 -> 90.5 mm
- net +5V: track 196.8 -> 157.9 mm
- net +11.1V: track 128.5 -> 105.3 mm
- net X_SHUT1: track 60.3 -> 75.2 mm, vias 0 -> 1
- net ENC_A: track 28.6 -> 13.9 mm
- net +5V_PI: track 38.8 -> 52.7 mm
- net ECHO1: track 40.8 -> 28.0 mm
- net ENC_B: track 32.9 -> 21.8 mm
- net ECHO3: track 29.7 -> 38.6 mm, vias 0 -> 1
- net SCL: track 92.4 -> 101.1 mm, vias 4 -> 0
- net TRIG3: track 37.4 -> 45.0 mm
- net SDA: track 95.7 -> 88.7 mm, vias 3 -> 1
- net X_SHUT2: track 57.6 -> 63.3 mm
- net XSHUT_4: track 48.8 -> 54.2 mm, vias 0 -> 1
- net +3V3: track 57.5 -> 62.5 mm, vias 0 -> 2
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