File: electrical/WRO_RevB_2/WRO_RevB_2.kicad_pcb (KiCad board)
At the start: 2 copper layers, 117.5 x 50.6 mm, 25 parts, among them J11 MOTOR, J2 Conn_01x04_Pin, J3 Conn_01x04_Pin, J4 Conn_01x11_Pin, J5 Conn_01x08_Pin, U2 ROB-14450

Commit message: actualiza PCB RevB
Parts:
- moved J11 20.2 mm to (157.4, 79.6), turned to 0 degrees
- moved US1 15.0 mm to (156.7, 105.8)
- moved R4 13.9 mm to (146.8, 89.1), turned to 180 degrees
- moved US3 13.8 mm to (156.7, 91.7)
- moved G*** 9.55 mm to (171.7, 81.8)
- moved R3 9.47 mm to (146.8, 84.3), turned to 180 degrees
- moved C5 6.12 mm to (136.8, 120.1)
- moved C6 6.12 mm to (142.9, 121.0)
- moved TOF3 4.70 mm to (143.4, 94.6)
- moved TOF4 4.59 mm to (143.4, 101.8)
- moved TOF1 4.00 mm to (130.8, 94.6)
- moved TOF2 3.87 mm to (130.8, 101.8)
- moved US2 2.74 mm to (156.7, 98.7)
Routing:
- net GND: track 90.5 -> 26.2 mm
- net +5V: track 157.9 -> 196.8 mm
- net +11.1V: track 105.3 -> 128.5 mm
- net X_SHUT1: track 75.2 -> 60.3 mm, vias 1 -> 0
- net ENC_A: track 13.9 -> 28.6 mm
- net +5V_PI: track 52.7 -> 38.8 mm
- net ECHO1: track 28.0 -> 40.8 mm
- net ENC_B: track 21.8 -> 32.9 mm
- net ECHO3: track 38.6 -> 29.7 mm, vias 1 -> 0
- net SCL: track 101.1 -> 92.4 mm, vias 0 -> 4
- net TRIG3: track 45.0 -> 37.4 mm
- net SDA: track 88.7 -> 95.7 mm, vias 1 -> 3
- net X_SHUT2: track 63.3 -> 57.6 mm
- net XSHUT_4: track 54.2 -> 48.8 mm, vias 1 -> 0
- net +3V3: track 62.5 -> 57.5 mm, vias 2 -> 0
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
Commit message: pcb done (again)
Parts:
- added N1: Housing, Symbol:KiCad-Logo2_12mm_SilkScreen, F.Cu at (15.2, 5.93)
Connections:
- TOF1 pad 3: SCL -> SDA
- TOF1 pad 4: SDA -> SCL
- TOF2 pad 3: SCL -> SDA
- TOF2 pad 4: SDA -> SCL
- TOF3 pad 3: SCL -> SDA
- TOF3 pad 4: SDA -> SCL
- TOF4 pad 3: SCL -> SDA
- TOF4 pad 4: SDA -> SCL
Routing:
- net SDA: track 95.7 -> 91.8 mm
- net SCL: track 92.4 -> 94.7 mm, vias 4 -> 3
